File: 007.kicad_sch (KiCad schematic)
At the start: 68 parts, among them U1 AM6232ASCGHAALWR

Commit message: Remove rando NCs added during conversion
Also a little tidying.

TODO: check junctions that may be missing. Noticed a few obvious ones
and corrected them already.

Signed-off-by: Michael Welling <mwelling79@gmail.com>
Connections:
- no-connect marks 134 -> 0
