File: 012.kicad_sch (KiCad schematic)
At the start: 1 part, among them U1 AM6232ASCGHAALWR

Commit message: Remove rando NCs added during conversion
Also a little tidying.

TODO: check junctions that may be missing. Noticed a few obvious ones
and corrected them already.

Signed-off-by: Michael Welling <mwelling79@gmail.com>
Other:
- moved on the sheet: U1J, U1M, U1S

Commit message: Another round of cleansing fire
Signed-off-by: Michael Welling <mwelling79@gmail.com>
Other:
- moved on the sheet: U1M, U1S
