File: 013.kicad_sch (KiCad schematic)
At the start: 3 parts, among them U1 AM6232ASCGHAALWR

Commit message: Remove rando NCs added during conversion
Also a little tidying.

TODO: check junctions that may be missing. Noticed a few obvious ones
and corrected them already.

Signed-off-by: Michael Welling <mwelling79@gmail.com>
Connections:
- no-connect marks 8 -> 4
Other:
- moved on the sheet: R25, R27, U1A

Commit message: Another round of cleansing fire
Signed-off-by: Michael Welling <mwelling79@gmail.com>
Changed lines of the file:
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@@
 		)
 		(property "Value" "AM6232ASCGHAALWR"
-			(at 20.32 250.444 0)
+			(at 33.274 249.936 0)
 			(effects
 				(font
@@
 		)
 		(property "PCB FOOTPRINT" "bga425_0d5_13x13mm"
-			(at 20.32 256.54 0)
+			(at 33.274 256.032 0)
 			(effects
 				(font
@@
 		)
 		(property "PACKAGE SIZE" "BGA425"
-			(at 20.32 253.746 0)
+			(at 33.274 253.238 0)
 			(effects
 				(font
@@
 		)
 		(property "Value" "AM6232ASCGHAALWR"
-			(at 15.24 172.72 0)
+			(at 32.766 172.72 0)
 			(effects
 				(font
@@
 		)
 		(property "PCB FOOTPRINT" "bga425_0d5_13x13mm"
-			(at 15.24 177.8 0)
+			(at 32.766 177.8 0)
 			(effects
 				(font
@@
 		)
 		(property "PACKAGE SIZE" "BGA425"
-			(at 15.24 175.26 0)
-			(effects
-				(font
+			(at 32.766 175.26 0)
+			(effects
+				(font
