File: 015.kicad_sch (KiCad schematic)
At the start: 41 parts, among them J1 TC2050-IDC, J4 3P-1.0mm, SW1 Tactile Switch, SW2 Tactile Switch, U1 AM6232ASCGHAALWR, U11 MSPM0L1105TRGER, U13 SN74LVC2G241DCUR

Commit message: Remove rando NCs added during conversion
Also a little tidying.

TODO: check junctions that may be missing. Noticed a few obvious ones
and corrected them already.

Signed-off-by: Michael Welling <mwelling79@gmail.com>
Connections:
- no-connect marks 37 -> 15
Other:
- moved on the sheet: SW1, SW2

Commit message: Another round of cleansing fire
Signed-off-by: Michael Welling <mwelling79@gmail.com>
Connections:
- no-connect marks 15 -> 5
Changed lines of the file:
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@@
-	)
-	(no_connect
-		(at 144.78 154.94)
-	)
-	(no_connect
-		(at 149.86 129.54)
-	)
-	(no_connect
-		(at 137.16 154.94)
 	)
 	(no_connect
@@
 	)
 	(no_connect
-		(at 162.56 129.54)
-	)
-	(no_connect
-		(at 121.92 154.94)
-	)
-	(no_connect
 		(at 66.04 134.62)
-	)
-	(no_connect
-		(at 114.3 154.94)
 	)
 	(no_connect
 		(at 66.04 129.54)
 	)
-	(no_connect
-		(at 149.86 154.94)
-	)
-	(no_connect
-		(at 127 154.94)
-	)
-	(no_connect
-		(at 157.48 154.94)
-	)
-	(no_connect
-		(at 134.62 154.94)
-	)
 	(wire
