File: 015.kicad_sch (KiCad schematic)
At the start: 41 parts, among them J1 TC2050-IDC, J4 3P-1.0mm, SW1 Tactile Switch, SW2 Tactile Switch, U1 AM6232ASCGHAALWR, U11 MSPM0L1105TRGER, U13 SN74LVC2G241DCUR

Commit message: Moar fixes
Mostly missing junctions flagged in review on discord.

Signed-off-by: Michael Welling <mwelling79@gmail.com>
Connections:
- net VDD_3V3: now also R33.1, R35.1
Changed lines of the file:
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@@
+	)
+	(junction
+		(at 353.06 33.02)
+		(diameter 0)
+		(color 0 0 0 0)
 	)
 	(junction
@@
 		(pts
 			(xy 294.64 53.34) (xy 289.56 53.34)
+		)
+		(stroke
+			(width 0)
+			(type default)
+		)
+	)
+	(wire
+		(pts
+			(xy 353.06 33.02) (xy 365.76 33.02)
 		)
 		(stroke
@@
 	(wire
 		(pts
-			(xy 353.06 38.1) (xy 353.06 30.48)
+			(xy 353.06 38.1) (xy 353.06 33.02)
 		)
 		(stroke
@@
 		(pts
 			(xy 66.04 147.32) (xy 53.34 147.32)
+		)
+		(stroke
+			(width 0)
+			(type default)
+		)
+	)
+	(wire
+		(pts
+			(xy 353.06 33.02) (xy 353.06 30.48)
 		)
 		(stroke
@@
 	(wire
 		(pts
-			(xy 340.36 33.02) (xy 365.76 33.02)
-		)
-		(stroke
+			(xy 340.36 33.02) (xy 353.06 33.02)
+		)
+		(stroke
