File: 005.kicad_sch (KiCad schematic)
At the start: 68 parts, among them U10 LM73100RPWR, U12 TLV62595DMQR, U17 TPS6521903RHBR, U5 BQ21040, U7 LM73100RPWR, U9 LM73100RPWR

Commit message: Remove rando NCs added during conversion
Also a little tidying.

TODO: check junctions that may be missing. Noticed a few obvious ones
and corrected them already.

Signed-off-by: Michael Welling <mwelling79@gmail.com>
Connections:
- net VDD_1V2: now also L17.2, TP21.1 (TP), U17.24 (FB_B3)
- net VDD_1V8: now also L16.2, TP20.1 (TP), U17.32 (FB_B2)
- no-connect marks 112 -> 10
Other:
- moved on the sheet: C10, C103, C11, C112, C113, C12, C125, C13, C133, C134, C135, C14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

Commit message: Moar fixes
Mostly missing junctions flagged in review on discord.

Signed-off-by: Michael Welling <mwelling79@gmail.com>
Connections:
- no-connect marks 10 -> 7
Changed lines of the file:
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@@
-	)
-	(no_connect
-		(at 288.29 203.2)
 	)
 	(no_connect
@@
 	)
 	(no_connect
-		(at 199.39 200.66)
-	)
-	(no_connect
 		(at 34.29 73.66)
 	)
@@
 		(at 189.23 73.66)
 	)
-	(no_connect
-		(at 191.77 200.66)
-	)
 	(wire
