File: 009.kicad_sch (KiCad schematic)
At the start: 57 parts, among them J3 ST-TF-MR267, U1 AM6232ASCGHAALWR, U3 EMMC04G-MT32-01G10, U8 TPS22918DBVR

Commit message: Remove rando NCs added during conversion
Also a little tidying.

TODO: check junctions that may be missing. Noticed a few obvious ones
and corrected them already.

Signed-off-by: Michael Welling <mwelling79@gmail.com>
Connections:
- no-connect marks 197 -> 141
Other:
- moved on the sheet: C33, C34, C35, D19, D2, D20, D21, D22, D23, D26, J3, R30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

Commit message: Another round of cleansing fire
Signed-off-by: Michael Welling <mwelling79@gmail.com>
Connections:
- net at D56.1 (A), R14.2, U3.K5 (RST_n): now also D47.1 (A), D48.1 (A)
- no-connect marks 141 -> 129
Changed lines of the file:
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@@
+	)
+	(junction
+		(at 226.06 101.6)
+		(diameter 0)
+		(color 0 0 0 0)
 	)
 	(junction
@@
 	)
 	(no_connect
-		(at 93.98 215.9)
-	)
-	(no_connect
 		(at 402.59 115.57)
 	)
@@
 	)
 	(no_connect
-		(at 311.15 238.76)
-	)
-	(no_connect
 		(at 361.95 41.91)
 	)
@@
 	)
 	(no_connect
-		(at 96.52 236.22)
-	)
-	(no_connect
 		(at 402.59 97.79)
 	)
@@
 	)
 	(no_connect
-		(at 306.07 238.76)
-	)
-	(no_connect
 		(at 402.59 74.93)
 	)
@@
 	)
 	(no_connect
-		(at 318.77 238.76)
-	)
-	(no_connect
 		(at 402.59 72.39)
 	)
@@
 	)
 	(no_connect
-		(at 323.85 238.76)
-	)
-	(no_connect
-		(at 81.28 215.9)
-	)
-	(no_connect
 		(at 361.95 130.81)
 	)
@@
 	)
 	(no_connect
-		(at 331.47 238.76)
-	)
-	(no_connect
 		(at 361.95 158.75)
 	)
@@
 	)
 	(no_connect
-		(at 144.78 238.76)
-	)
-	(no_connect
 		(at 402.59 90.17)
 	)
@@
 	)
 	(no_connect
-		(at 298.45 238.76)
-	)
-	(no_connect
-		(at 104.14 236.22)
-	)
-	(no_connect
 		(at 361.95 39.37)
 	)
@@
 	(no_connect
 		(at 361.95 69.85)
-	)
-	(no_connect
-		(at 152.4 238.76)
 	)
 	(no_connect
@@
 	(wire
 		(pts
-			(xy 220.98 101.6) (xy 246.38 101.6)
+			(xy 220.98 101.6) (xy 226.06 101.6)
 		)
 		(stroke
@@
 	(wire
 		(pts
+			(xy 226.06 101.6) (xy 246.38 101.6)
+		)
+		(stroke
+			(width 0)
+			(type default)
+		)
+	)
+	(wire
+		(pts
 			(xy 154.94 25.4) (xy 154.94 20.32)
 		)
@@
 	(wire
 		(pts
-			(xy 226.06 109.22) (xy 226.06 93.98)
+			(xy 226.06 109.22) (xy 226.06 101.6)
 		)
 		(stroke
@@
 		)
 		(stroke
+			(width 0)
+			(type default)
+		)
+	)
+	(wire
+		(pts
+			(xy 226.06 101.6) (xy 226.06 93.98)
+		)
+		(stroke

Commit message: Moar fixes
Mostly missing junctions flagged in review on discord.

Signed-off-by: Michael Welling <mwelling79@gmail.com>
Connections:
- net SD_CLK: now also D22.2, R90.2
- net SD_CMD: now also D21.2, R89.2
- net SD_D0: now also D23.2, R92.2
- net SD_D1: now also D26.2, R95.2
- net SD_D2: now also D19.2, R79.2
Changed lines of the file:
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@@
 	)
 	(junction
+		(at 293.37 223.52)
+		(diameter 0)
+		(color 0 0 0 0)
+	)
+	(junction
 		(at 246.38 101.6)
 		(diameter 0)
@@
 	)
 	(junction
+		(at 267.97 215.9)
+		(diameter 0)
+		(color 0 0 0 0)
+	)
+	(junction
 		(at 185.42 20.32)
 		(diameter 0)
@@
 	)
 	(junction
+		(at 280.67 220.98)
+		(diameter 0)
+		(color 0 0 0 0)
+	)
+	(junction
 		(at 205.74 20.32)
 		(diameter 0)
@@
 	)
 	(junction
+		(at 229.87 205.74)
+		(diameter 0)
+		(color 0 0 0 0)
+	)
+	(junction
 		(at 124.46 246.38)
 		(diameter 0)
@@
 		(color 0 0 0 0)
 	)
+	(junction
+		(at 255.27 210.82)
+		(diameter 0)
+		(color 0 0 0 0)
+	)
 	(no_connect
 		(at 317.5 132.08)
@@
 	(wire
 		(pts
-			(xy 171.45 210.82) (xy 344.17 210.82)
+			(xy 171.45 210.82) (xy 255.27 210.82)
 		)
 		(stroke
@@
 	(wire
 		(pts
-			(xy 171.45 220.98) (xy 344.17 220.98)
+			(xy 171.45 220.98) (xy 280.67 220.98)
 		)
 		(stroke
@@
 	(wire
 		(pts
+			(xy 229.87 205.74) (xy 344.17 205.74)
+		)
+		(stroke
+			(width 0)
+			(type default)
+		)
+	)
+	(wire
+		(pts
 			(xy 389.89 218.44) (xy 389.89 215.9)
 		)
@@
 	(wire
 		(pts
-			(xy 171.45 215.9) (xy 344.17 215.9)
+			(xy 171.45 215.9) (xy 267.97 215.9)
 		)
 		(stroke
@@
 	(wire
 		(pts
-			(xy 267.97 228.6) (xy 267.97 195.58)
+			(xy 267.97 228.6) (xy 267.97 215.9)
 		)
 		(stroke
@@
 	(wire
 		(pts
-			(xy 255.27 228.6) (xy 255.27 195.58)
+			(xy 255.27 228.6) (xy 255.27 210.82)
 		)
 		(stroke
@@
 	(wire
 		(pts
+			(xy 280.67 220.98) (xy 280.67 195.58)
+		)
+		(stroke
+			(width 0)
+			(type default)
+		)
+	)
+	(wire
+		(pts
 			(xy 154.94 25.4) (xy 154.94 20.32)
 		)
@@
 	(wire
 		(pts
+			(xy 280.67 220.98) (xy 344.17 220.98)
+		)
+		(stroke
+			(width 0)
+			(type default)
+		)
+	)
+	(wire
+		(pts
 			(xy 353.06 63.5) (xy 353.06 58.42)
 		)
@@
 	(wire
 		(pts
+			(xy 293.37 223.52) (xy 293.37 195.58)
+		)
+		(stroke
+			(width 0)
+			(type default)
+		)
+	)
+	(wire
+		(pts
 			(xy 217.17 246.38) (xy 229.87 246.38)
 		)
@@
 	(wire
 		(pts
+			(xy 255.27 210.82) (xy 344.17 210.82)
+		)
+		(stroke
+			(width 0)
+			(type default)
+		)
+	)
+	(wire
+		(pts
 			(xy 208.28 101.6) (xy 203.2 101.6)
 		)
@@
 	(wire
 		(pts
-			(xy 280.67 228.6) (xy 280.67 195.58)
+			(xy 280.67 228.6) (xy 280.67 220.98)
 		)
 		(stroke
@@
 	(wire
 		(pts
-			(xy 171.45 205.74) (xy 344.17 205.74)
+			(xy 171.45 205.74) (xy 229.87 205.74)
 		)
 		(stroke
@@
 	(wire
 		(pts
-			(xy 293.37 228.6) (xy 293.37 195.58)
+			(xy 293.37 228.6) (xy 293.37 223.52)
+		)
+		(stroke
+			(width 0)
+			(type default)
+		)
+	)
+	(wire
+		(pts
+			(xy 293.37 223.52) (xy 344.17 223.52)
 		)
 		(stroke
@@
 	(wire
 		(pts
+			(xy 267.97 215.9) (xy 267.97 195.58)
+		)
+		(stroke
+			(width 0)
+			(type default)
+		)
+	)
+	(wire
+		(pts
 			(xy 124.46 246.38) (xy 149.86 246.38)
 		)
@@
 	(wire
 		(pts
+			(xy 255.27 210.82) (xy 255.27 195.58)
+		)
+		(stroke
+			(width 0)
+			(type default)
+		)
+	)
+	(wire
+		(pts
 			(xy 328.93 233.68) (xy 328.93 213.36)
 		)
@@
 	(wire
 		(pts
-			(xy 229.87 228.6) (xy 229.87 195.58)
+			(xy 229.87 228.6) (xy 229.87 205.74)
 		)
 		(stroke
@@
 	(wire
 		(pts
-			(xy 171.45 223.52) (xy 344.17 223.52)
+			(xy 171.45 223.52) (xy 293.37 223.52)
 		)
 		(stroke
@@
 	(wire
 		(pts
+			(xy 229.87 205.74) (xy 229.87 195.58)
+		)
+		(stroke
+			(width 0)
+			(type default)
+		)
+	)
+	(wire
+		(pts
 			(xy 316.23 243.84) (xy 303.53 243.84)
 		)
@@
 	(wire
 		(pts
+			(xy 267.97 215.9) (xy 344.17 215.9)
+		)
+		(stroke
+			(width 0)
+			(type default)
+		)
+	)
+	(wire
+		(pts
 			(xy 91.44 76.2) (xy 236.22 76.2)
 		)
@@
 		(dnp no)
 		(property "Reference" "U1"
-			(at 7.62 44.45 0)
+			(at 12.954 44.958 0)
 			(effects
 				(font
