File: 014.kicad_sch (KiCad schematic)
At the start: 19 parts, among them J14 USB2.0 Type C, U1 AM6232ASCGHAALWR, U6 TVS0500DRVR

Commit message: Moar fixes
Mostly missing junctions flagged in review on discord.

Signed-off-by: Michael Welling <mwelling79@gmail.com>
Changed lines of the file:
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@@
 		)
 		(property "Value" "AM6232ASCGHAALWR"
-			(at 28.448 250.19 0)
+			(at 32.766 249.936 0)
 			(effects
 				(font
@@
 		)
 		(property "PCB FOOTPRINT" "bga425_0d5_13x13mm"
-			(at 28.448 256.286 0)
+			(at 32.766 256.032 0)
 			(effects
 				(font
@@
 		)
 		(property "PACKAGE SIZE" "BGA425"
-			(at 28.448 253.492 0)
+			(at 32.766 253.238 0)
 			(effects
 				(font
